Commit message: added urdf for gundam (PR2 + Roman)

File: src/roman_model/urdf/roman_body.urdf.xacro (robot description, xacro)
@@ -4,11 +4,11 @@
     <xacro:include filename="$(find roman_model)/control/roman_body.transmission.xacro"/>
     <xacro:include filename="$(find hector_sensors_description)/urdf/asus_camera.urdf.xacro"/>
-    <xacro:macro name="roman_body" params="name parent *origin namespace">
-        <joint name="torso_joint0" type="fixed">
-            <parent link="${parent}"/>
-            <child link="torso_link0"/>
+    <xacro:macro name="roman_body" params="name parent *origin namespace prefix">
+        <joint name="${prefix}torso_joint0" type="fixed">
+            <parent link="${prefix}${parent}"/>
+            <child link="${prefix}torso_link0"/>
             <insert_block name="origin"/>
         </joint>
-        <link name="torso_link0">
+        <link name="${prefix}torso_link0">
             <!-- dummy inertial values -->
             <inertial>
@@ -39,13 +39,13 @@
             </collision>
         </link>
-        <joint name="torso_joint1" type="revolute">
+        <joint name="${prefix}torso_joint1" type="revolute">
             <origin xyz="0.593 0 0" rpy="3.14159 0 0"/>
             <axis xyz="1 0 0"/>
-            <parent link="torso_link0"/>
-            <child link="chest"/>
+            <parent link="${prefix}torso_link0"/>
+            <child link="${prefix}chest"/>
             <limit effort="1000.0" lower="-6.283185" upper="6.283185" velocity="0.5"/>
             <dynamics damping="1.0" friction="10.0"/>
         </joint>
-        <link name="chest">
+        <link name="${prefix}chest">
             <inertial>
                 <mass value="10.0"/>
@@ -71,5 +71,5 @@
             </collision>
         </link>
-        <xacro:asus_camera name="asus" parent="chest">
+        <xacro:asus_camera name="${prefix}asus" parent="${prefix}chest">
             <origin xyz="0.05 -0.075 0" rpy="${-M_PI/2} 0.0 -2.09"/>
         </xacro:asus_camera>

File: src/roman_model/urdf/talon.urdf.xacro (robot description, xacro)
@@ -4,18 +4,18 @@
     <xacro:include filename="$(find roman_model)/control/talon.transmission.xacro"/>
     <xacro:include filename="$(find hector_sensors_description)/urdf/hokuyo_utm30lx.urdf.xacro"/>
-    <xacro:macro name="talon" params="name namespace">
-        <link name="${name}_footprint"/>
-        <joint name="${name}_footprint_joint" type="fixed">
+    <xacro:macro name="talon" params="name namespace prefix">
+        <link name="${prefix}${name}_footprint"/>
+        <joint name="${prefix}${name}_footprint_joint" type="fixed">
             <origin xyz="0 0 0.15203" rpy="0 0 0"/>
-            <parent link="${name}_footprint"/>
-            <child link="${name}_link"/>
+            <parent link="${prefix}${name}_footprint"/>
+            <child link="${prefix}${name}_link"/>
         </joint>
-        <link name="${name}_link"/>
-        <joint name="${name}_joint" type="fixed">
+        <link name="${prefix}${name}_link"/>
+        <joint name="${prefix}${name}_joint" type="fixed">
             <origin xyz="0 0 0" rpy="3.14 0 0"/>
-            <parent link="${name}_link"/>
-            <child link="talon"/>
+            <parent link="${prefix}${name}_link"/>
+            <child link="${prefix}talon"/>
         </joint>
-        <link name="talon">
+        <link name="${prefix}talon">
             <inertial>
                 <mass value="40.0"/>
@@ -64,16 +64,16 @@
             </collision>
         </link>
-        <xacro:hokuyo_utm30lx_gpu name="base_laser" parent="base_link" ros_topic="base_scan" update_rate="20.0" ray_count="1080" min_angle="-130" max_angle="130">
+        <xacro:hokuyo_utm30lx_gpu name="${prefix}base_laser" parent="${prefix}base_link" ros_topic="base_scan" update_rate="20.0" ray_count="1080" min_angle="-130" max_angle="130">
             <origin xyz="0.50 0 0.210" rpy="0 0 0"/>
         </xacro:hokuyo_utm30lx_gpu>
-        <joint name="track_left_joint" type="revolute">
+        <joint name="${prefix}track_left_joint" type="revolute">
             <origin xyz="0.000000 0.000000 0.000000" rpy="0 0 0"/>
             <axis xyz="0 0 1"/>
-            <parent link="talon"/>
-            <child link="track_left"/>
+            <parent link="${prefix}talon"/>
+            <child link="${prefix}track_left"/>
             <limit effort="1000.0" lower="-3.141593" upper="3.141593" velocity="0.5"/>
             <dynamics damping="0.0" friction="0.0"/>
         </joint>
-        <link name="track_left">
+        <link name="${prefix}track_left">
             <!-- dummy inertial values -->
             <inertial>
@@ -83,13 +83,13 @@
             </inertial>
         </link>
-        <joint name="track_right_joint" type="revolute">
+        <joint name="${prefix}track_right_joint" type="revolute">
             <origin xyz="0.000000 0.000000 0.000000" rpy="0 0 0"/>
             <axis xyz="0 0 1"/>
-            <parent link="talon"/>
-            <child link="track_right"/>
+            <parent link="${prefix}talon"/>
+            <child link="${prefix}track_right"/>
             <limit effort="1000.0" lower="-3.141593" upper="3.141593" velocity="0.5"/>
             <dynamics damping="0.0" friction="0.0"/>
         </joint>
-        <link name="track_right">
+        <link name="${prefix}track_right">
             <!-- dummy inertial values -->
             <inertial>
