Commit message: reverted fully to origin roman_model

File: src/roman_model/urdf/talon.urdf.xacro (robot description, xacro)
@@ -4,18 +4,18 @@
     <xacro:include filename="$(find roman_model)/control/talon.transmission.xacro"/>
     <xacro:include filename="$(find hector_sensors_description)/urdf/hokuyo_utm30lx.urdf.xacro"/>
-    <xacro:macro name="talon" params="name namespace prefix">
-        <link name="${prefix}${name}_footprint"/>
-        <joint name="${prefix}${name}_footprint_joint" type="fixed">
+    <xacro:macro name="talon" params="name namespace">
+        <link name="${name}_footprint"/>
+        <joint name="${name}_footprint_joint" type="fixed">
             <origin xyz="0 0 0.15203" rpy="0 0 0"/>
-            <parent link="${prefix}${name}_footprint"/>
-            <child link="${prefix}${name}_link"/>
+            <parent link="${name}_footprint"/>
+            <child link="${name}_link"/>
         </joint>
-        <link name="${prefix}${name}_link"/>
-        <joint name="${prefix}${name}_joint" type="fixed">
+        <link name="${name}_link"/>
+        <joint name="${name}_joint" type="fixed">
             <origin xyz="0 0 0" rpy="3.14 0 0"/>
-            <parent link="${prefix}${name}_link"/>
-            <child link="${prefix}talon"/>
+            <parent link="${name}_link"/>
+            <child link="talon"/>
         </joint>
-        <link name="${prefix}talon">
+        <link name="talon">
             <inertial>
                 <mass value="40.0"/>
@@ -64,16 +64,16 @@
             </collision>
         </link>
-        <xacro:hokuyo_utm30lx_gpu name="${prefix}base_laser" parent="${prefix}base_link" ros_topic="base_scan" update_rate="20.0" ray_count="1080" min_angle="-130" max_angle="130">
+        <xacro:hokuyo_utm30lx_gpu name="base_laser" parent="base_link" ros_topic="base_scan" update_rate="20.0" ray_count="1080" min_angle="-130" max_angle="130">
             <origin xyz="0.50 0 0.210" rpy="0 0 0"/>
         </xacro:hokuyo_utm30lx_gpu>
-        <joint name="${prefix}track_left_joint" type="revolute">
+        <joint name="track_left_joint" type="revolute">
             <origin xyz="0.000000 0.000000 0.000000" rpy="0 0 0"/>
             <axis xyz="0 0 1"/>
-            <parent link="${prefix}talon"/>
-            <child link="${prefix}track_left"/>
+            <parent link="talon"/>
+            <child link="track_left"/>
             <limit effort="1000.0" lower="-3.141593" upper="3.141593" velocity="0.5"/>
             <dynamics damping="0.0" friction="0.0"/>
         </joint>
-        <link name="${prefix}track_left">
+        <link name="track_left">
             <!-- dummy inertial values -->
             <inertial>
@@ -83,13 +83,13 @@
             </inertial>
         </link>
-        <joint name="${prefix}track_right_joint" type="revolute">
+        <joint name="track_right_joint" type="revolute">
             <origin xyz="0.000000 0.000000 0.000000" rpy="0 0 0"/>
             <axis xyz="0 0 1"/>
-            <parent link="${prefix}talon"/>
-            <child link="${prefix}track_right"/>
+            <parent link="talon"/>
+            <child link="track_right"/>
             <limit effort="1000.0" lower="-3.141593" upper="3.141593" velocity="0.5"/>
             <dynamics damping="0.0" friction="0.0"/>
         </joint>
-        <link name="${prefix}track_right">
+        <link name="track_right">
             <!-- dummy inertial values -->
             <inertial>
