Commit message: gripper fake joint server created, included large cube collision object for bookshelf

File: src/gundam_description/urdf/gundam.urdf.xacro (robot description, xacro)
@@ -27,5 +27,5 @@
    </joint>
   <joint name="world_joint_pr2" type="fixed">
-      <origin xyz="0 1.5 0"  rpy="0 0 0" />
+      <origin xyz="0 2.25 0"  rpy="0 0 0" />
       <parent link="world_link" />
       <child link="pr2/base_footprint" />
@@ -120,5 +120,6 @@
     <xacro:include filename="$(find roman_model)/urdf/talon.urdf.xacro"/>
     <xacro:include filename="$(find roman_model)/urdf/roman_body.urdf.xacro"/>
-    <xacro:include filename="$(find roman_model)/urdf/robosimian_arm.urdf.xacro"/>
+    <!-- Note: using joint limited (-1.57, 1.57) robosimian arm model -->
+    <xacro:include filename="$(find roman_model)/urdf/robosimian_arm_joint_limited.urdf.xacro"/>
     <xacro:include filename="$(find roman_model)/gazebo/gazebo.urdf.xacro"/>
     <xacro:talon name="base" namespace="$(arg namespace)" prefix="roman/"/>

Commit message: prefixing corrections. added velocities to sbpl trajectories in move arm server'

File: src/gundam_description/urdf/gundam.urdf.xacro (robot description, xacro)
@@ -24,10 +24,10 @@
       <origin xyz="0 0 0"  rpy="0 0 1.57" />
       <parent link="world_link" />
-      <child link="roman/base_footprint" />
+      <child link="roman_base_footprint" />
    </joint>
   <joint name="world_joint_pr2" type="fixed">
       <origin xyz="0 2.25 0"  rpy="0 0 0" />
       <parent link="world_link" />
-      <child link="pr2/base_footprint" />
+      <child link="pr2_base_footprint" />
    </joint>
 <!-- PR2 -->
@@ -67,20 +67,20 @@
        the origin block defines where the component is w.r.t its parent (in this case the parent
        is the world frame). For more, see http://www.ros.org/wiki/xacro -->
-  <xacro:pr2_base_v0 name="base" prefix="pr2/"/>
-  <xacro:pr2_torso_v0 name="torso_lift" parent="base_link" prefix="pr2/" >
+  <xacro:pr2_base_v0 name="base" prefix="pr2_"/>
+  <xacro:pr2_torso_v0 name="torso_lift" parent="base_link" prefix="pr2_" >
     <origin xyz="-0.05 0 0.739675" rpy="0 0 0" />
   </xacro:pr2_torso_v0>
-  <xacro:pr2_head_v0 name="head" parent="torso_lift_link" prefix="pr2/">
+  <xacro:pr2_head_v0 name="head" parent="torso_lift_link" prefix="pr2_">
     <origin xyz="-0.01707 0.0 0.38145"
             rpy="0.0 0.0 0.0" />
   </xacro:pr2_head_v0>
-  <xacro:pr2_shoulder_v0 side="r" reflect="-1" parent="torso_lift_link" prefix="pr2/">
+  <xacro:pr2_shoulder_v0 side="r" reflect="-1" parent="torso_lift_link" prefix="pr2_">
     <origin xyz="0.0 -0.188 0.0" rpy="0 0 0" />
   </xacro:pr2_shoulder_v0>
-  <xacro:pr2_upper_arm_v0 side="r" reflect="-1" parent="r_upper_arm_roll_link" prefix="pr2/" />
-  <xacro:pr2_forearm_v0 side="r" reflect="-1" parent="r_forearm_roll_link" prefix="pr2/">
+  <xacro:pr2_upper_arm_v0 side="r" reflect="-1" parent="r_upper_arm_roll_link" prefix="pr2_" />
+  <xacro:pr2_forearm_v0 side="r" reflect="-1" parent="r_forearm_roll_link" prefix="pr2_">
     <origin xyz="0 0 0" rpy="0 0 0" />
   </xacro:pr2_forearm_v0>
-  <xacro:pr2_gripper_v0 reflect="-1.0" side="r" parent="r_wrist_roll_link" prefix="pr2/"
+  <xacro:pr2_gripper_v0 reflect="-1.0" side="r" parent="r_wrist_roll_link" prefix="pr2_"
                screw_reduction="${4.0/1000.0}"
                gear_ratio="${(729.0/25.0)*(22.0/16.0)}"
@@ -96,12 +96,12 @@
   </xacro:pr2_gripper_v0>
   <!-- Optionally include left arm -->
-   <xacro:pr2_shoulder_v0 side="l" reflect="1" parent="torso_lift_link" prefix="pr2/" >
+   <xacro:pr2_shoulder_v0 side="l" reflect="1" parent="torso_lift_link" prefix="pr2_" >
     <origin xyz="0.0 0.188 0.0" rpy="0 0 0" />
   </xacro:pr2_shoulder_v0>
-  <xacro:pr2_upper_arm_v0 side="l" reflect="1" parent="l_upper_arm_roll_link" prefix="pr2/" />
-  <xacro:pr2_forearm_v0 side="l" reflect="1" parent="l_forearm_roll_link" prefix="pr2/" >
+  <xacro:pr2_upper_arm_v0 side="l" reflect="1" parent="l_upper_arm_roll_link" prefix="pr2_" />
+  <xacro:pr2_forearm_v0 side="l" reflect="1" parent="l_forearm_roll_link" prefix="pr2_" >
     <origin xyz="0 0 0" rpy="0 0 0" />
   </xacro:pr2_forearm_v0>
-  <xacro:pr2_gripper_v0 reflect="1.0" side="l" parent="l_wrist_roll_link" prefix="pr2/"
+  <xacro:pr2_gripper_v0 reflect="1.0" side="l" parent="l_wrist_roll_link" prefix="pr2_"
                screw_reduction="${4.0/1000.0}"
                gear_ratio="${(729.0/25.0)*(22.0/16.0)}"
@@ -123,14 +123,14 @@
     <xacro:include filename="$(find roman_model)/urdf/robosimian_arm_joint_limited.urdf.xacro"/>
     <xacro:include filename="$(find roman_model)/gazebo/gazebo.urdf.xacro"/>
-    <xacro:talon name="base" namespace="$(arg namespace)" prefix="roman/"/>
-    <xacro:roman_body name="roman_body" parent="talon" namespace="$(arg namespace)" prefix="roman/" >
+    <xacro:talon name="base" namespace="$(arg namespace)" prefix="roman_"/>
+    <xacro:roman_body name="roman_body" parent="talon" namespace="$(arg namespace)" prefix="roman_" >
         <origin xyz="0.355000 0.000000 0.090000" rpy="3.141592 1.570800 1.570800"/>
     </xacro:roman_body>
     <!--
-    <xacro:robosimian_arm prefix="roman/limb_left_" parent="roman/chest" namespace="$(arg namespace)">
+    <xacro:robosimian_arm prefix="roman_limb_left_" parent="roman_chest" namespace="$(arg namespace)">
         <origin xyz="0.0705 0.025 -0.1" rpy="0 1.5708 -1.5708"/>
     </xacro:robosimian_arm>
     -->
-    <xacro:robosimian_arm prefix="roman/limb_right_" parent="roman/chest" namespace="$(arg namespace)">
+    <xacro:robosimian_arm prefix="roman_limb_right_" parent="roman_chest" namespace="$(arg namespace)">
         <origin xyz="0.0705 0.025 0.1" rpy="0 -1.57080 -1.5708"/>
     </xacro:robosimian_arm>

File: src/pr2_description/robots/pr2_namespaced.urdf.xacro (robot description, xacro)
@@ -33,5 +33,5 @@
   <xacro:include filename="$(find pr2_description)/urdf/materials.urdf.xacro" />
   <!-- Included to put PR2 links and joints into its own namespace -->
-  <xacro:arg name="namespace" default="pr2/"/>
+  <xacro:arg name="namespace" default="pr2_"/>
   <!-- Now we can start using the macros included above to define the actual PR2 -->
   <!-- The first use of a macro.  This one was defined in base.urdf.xacro above.

Commit message: moved modified roman URDF files to gundam_description to avoid future conflicts

File: src/gundam_description/urdf/gundam.urdf.xacro (robot description, xacro)
@@ -118,9 +118,9 @@
   <!-- ROMAN -->
     <xacro:arg name="namespace" default="false" />
-    <xacro:include filename="$(find roman_model)/urdf/talon.urdf.xacro"/>
-    <xacro:include filename="$(find roman_model)/urdf/roman_body.urdf.xacro"/>
+    <xacro:include filename="$(find gundam_description)/urdf/talon.urdf.xacro"/>
+    <xacro:include filename="$(find gundam_description)/urdf/roman_body.urdf.xacro"/>
     <!-- Note: using joint limited (-1.57, 1.57) robosimian arm model -->
-    <xacro:include filename="$(find roman_model)/urdf/robosimian_arm_joint_limited.urdf.xacro"/>
-    <xacro:include filename="$(find roman_model)/gazebo/gazebo.urdf.xacro"/>
+    <xacro:include filename="$(find gundam_description)/urdf/robosimian_arm_joint_limited.urdf.xacro"/>
+    <xacro:include filename="$(find gundam_description)/gazebo/gazebo.urdf.xacro"/>
     <xacro:talon name="base" namespace="$(arg namespace)" prefix="roman/"/>
     <xacro:roman_body name="roman_body" parent="talon" namespace="$(arg namespace)" prefix="roman/" >

File: src/gundam_description/urdf/roman_body.urdf.xacro (robot description, xacro)
@@ -4,11 +4,11 @@
     <xacro:include filename="$(find roman_model)/control/roman_body.transmission.xacro"/>
     <xacro:include filename="$(find hector_sensors_description)/urdf/asus_camera.urdf.xacro"/>
-    <xacro:macro name="roman_body" params="name parent *origin namespace">
-        <joint name="torso_joint0" type="fixed">
-            <parent link="${parent}"/>
-            <child link="torso_link0"/>
+    <xacro:macro name="roman_body" params="name parent *origin namespace prefix">
+        <joint name="${prefix}torso_joint0" type="fixed">
+            <parent link="${prefix}${parent}"/>
+            <child link="${prefix}torso_link0"/>
             <insert_block name="origin"/>
         </joint>
-        <link name="torso_link0">
+        <link name="${prefix}torso_link0">
             <!-- dummy inertial values -->
             <inertial>
@@ -39,16 +39,13 @@
             </collision>
         </link>
-        <joint name="torso_joint1" type="revolute">
+        <joint name="${prefix}torso_joint1" type="revolute">
             <origin xyz="0.593 0 0" rpy="3.14159 0 0"/>
             <axis xyz="1 0 0"/>
-            <parent link="torso_link0"/>
-            <child link="chest"/>
-<!--
+            <parent link="${prefix}torso_link0"/>
+            <child link="${prefix}chest"/>
             <limit effort="1000.0" lower="-6.283185" upper="6.283185" velocity="0.5"/>
--->
-            <limit effort="1000.0" lower="-0.436" upper="0.785" velocity="0.5"/>
             <dynamics damping="1.0" friction="10.0"/>
         </joint>
-        <link name="chest">
+        <link name="${prefix}chest">
             <inertial>
                 <mass value="10.0"/>
@@ -73,20 +70,6 @@
                 </geometry>
             </collision>
-            <!-- asus and stuff -->
-            <collision>
-                <origin xyz="0.05 -0.1645 0.03825" rpy="0 0 0"/>
-                <geometry>
-                    <box size="0.14 0.10609 0.14"/>
-                </geometry>
-            </collision>
-            <!-- hat -->
-            <collision>
-                <origin xyz="0.20 0.03 0.0"/>
-                <geometry>
-                    <box size="0.1 0.16 0.40"/>
-                </geometry>
-            </collision>
         </link>
-        <xacro:asus_camera name="asus" parent="chest">
+        <xacro:asus_camera name="${prefix}asus" parent="${prefix}chest">
             <origin xyz="0.05 -0.075 0" rpy="${-M_PI/2} 0.0 -2.09"/>
         </xacro:asus_camera>
